File: kicad/bloombot/bloombot.kicad_sch (KiCad schematic)
At the start: 14 parts, among them M1 Water valve 1, M2 Water valve 2, M3 Water valve 3, M4 Water valve 4, M5 Water valve 5, M6 Water valve 6, M7 Water valve 7, M8 Water valve 8, U1 Meanwell LRS-75-12, U2 LM2596, U3 LM2596, U4 Raspberry Pi Zero W, U6 DHT22

Commit message: feat: rename project to BloomBot
Other:
- title: Floraflow wiring schematic -> BloomBot wiring schematic
Changed lines of the file:
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@@
 	(paper "A4")
 	(title_block
-		(title "Floraflow wiring schematic")
+		(title "BloomBot wiring schematic")
 		(date "2026-06-30")
 		(rev "1.0")
@@
 		)
 		(instances
-			(project "floraflow"
+			(project "bloombot"
 				(path "/f8ca57fe-b4ec-4658-84e8-4883faa41e21"
 					(reference "#PWR05")
@@
 		)
 		(instances
-			(project "floraflow"
+			(project "bloombot"
 				(path "/f8ca57fe-b4ec-4658-84e8-4883faa41e21"
 					(reference "M3")
@@
 		)
 		(instances
-			(project "floraflow"
+			(project "bloombot"
 				(path "/f8ca57fe-b4ec-4658-84e8-4883faa41e21"
 					(reference "#PWR018")
@@
 		)
 		(instances
-			(project "floraflow"
+			(project "bloombot"
 				(path "/f8ca57fe-b4ec-4658-84e8-4883faa41e21"
 					(reference "#PWR01")
@@
 		)
 		(instances
-			(project "floraflow"
+			(project "bloombot"
 				(path "/f8ca57fe-b4ec-4658-84e8-4883faa41e21"
 					(reference "#PWR09")
@@
 		)
 		(instances
-			(project "floraflow"
+			(project "bloombot"
 				(path "/f8ca57fe-b4ec-4658-84e8-4883faa41e21"
 					(reference "#PWR016")
@@
 		)
 		(instances
-			(project "floraflow"
+			(project "bloombot"
 				(path "/f8ca57fe-b4ec-4658-84e8-4883faa41e21"
 					(reference "#PWR013")
@@
 		)
 		(instances
-			(project "floraflow"
+			(project "bloombot"
 				(path "/f8ca57fe-b4ec-4658-84e8-4883faa41e21"
 					(reference "U4")
@@
 		)
 		(instances
-			(project "floraflow"
+			(project "bloombot"
 				(path "/f8ca57fe-b4ec-4658-84e8-4883faa41e21"
 					(reference "#PWR06")
@@
 		)
 		(instances
-			(project "floraflow"
+			(project "bloombot"
 				(path "/f8ca57fe-b4ec-4658-84e8-4883faa41e21"
 					(reference "U2")
@@
 		)
 		(instances
-			(project "floraflow"
+			(project "bloombot"
 				(path "/f8ca57fe-b4ec-4658-84e8-4883faa41e21"
 					(reference "#PWR02")
@@
 		)
 		(instances
-			(project "floraflow"
+			(project "bloombot"
 				(path "/f8ca57fe-b4ec-4658-84e8-4883faa41e21"
 					(reference "#PWR017")
@@
 		)
 		(instances
-			(project "floraflow"
+			(project "bloombot"
 				(path "/f8ca57fe-b4ec-4658-84e8-4883faa41e21"
 					(reference "#PWR07")
@@
 		)
 		(instances
-			(project "floraflow"
+			(project "bloombot"
 				(path "/f8ca57fe-b4ec-4658-84e8-4883faa41e21"
 					(reference "#PWR08")
@@
 		)
 		(instances
-			(project "floraflow"
+			(project "bloombot"
 				(path "/f8ca57fe-b4ec-4658-84e8-4883faa41e21"
 					(reference "U6")
@@
 		)
 		(instances
-			(project "floraflow"
+			(project "bloombot"
 				(path "/f8ca57fe-b4ec-4658-84e8-4883faa41e21"
 					(reference "M5")
@@
 		)
 		(instances
-			(project "floraflow"
+			(project "bloombot"
 				(path "/f8ca57fe-b4ec-4658-84e8-4883faa41e21"
 					(reference "M7")
@@
 		)
 		(instances
-			(project "floraflow"
+			(project "bloombot"
 				(path "/f8ca57fe-b4ec-4658-84e8-4883faa41e21"
 					(reference "M8")
@@
 		)
 		(instances
-			(project "floraflow"
+			(project "bloombot"
 				(path "/f8ca57fe-b4ec-4658-84e8-4883faa41e21"
 					(reference "U3")
@@
 		)
 		(instances
-			(project "floraflow"
+			(project "bloombot"
 				(path "/f8ca57fe-b4ec-4658-84e8-4883faa41e21"
 					(reference "#PWR04")
@@
 		)
 		(instances
-			(project "floraflow"
+			(project "bloombot"
 				(path "/f8ca57fe-b4ec-4658-84e8-4883faa41e21"
 					(reference "#PWR020")
@@
 		)
 		(instances
-			(project "floraflow"
+			(project "bloombot"
 				(path "/f8ca57fe-b4ec-4658-84e8-4883faa41e21"
 					(reference "M6")
@@
 		)
 		(instances
-			(project "floraflow"
+			(project "bloombot"
 				(path "/f8ca57fe-b4ec-4658-84e8-4883faa41e21"
 					(reference "#PWR019")
@@
 		)
 		(instances
-			(project "floraflow"
+			(project "bloombot"
 				(path "/f8ca57fe-b4ec-4658-84e8-4883faa41e21"
 					(reference "#PWR012")
@@
 		)
 		(instances
-			(project "floraflow"
+			(project "bloombot"
 				(path "/f8ca57fe-b4ec-4658-84e8-4883faa41e21"
 					(reference "M2")
@@
 		)
 		(instances
-			(project "floraflow"
+			(project "bloombot"
 				(path "/f8ca57fe-b4ec-4658-84e8-4883faa41e21"
 					(reference "M4")
@@
 		)
 		(instances
-			(project "floraflow"
+			(project "bloombot"
 				(path "/f8ca57fe-b4ec-4658-84e8-4883faa41e21"
 					(reference "U5")
@@
 		)
 		(instances
-			(project "floraflow"
+			(project "bloombot"
 				(path "/f8ca57fe-b4ec-4658-84e8-4883faa41e21"
 					(reference "#PWR014")
@@
 		)
 		(instances
-			(project "floraflow"
+			(project "bloombot"
 				(path "/f8ca57fe-b4ec-4658-84e8-4883faa41e21"
 					(reference "#PWR03")
@@
 		)
 		(instances
-			(project "floraflow"
+			(project "bloombot"
 				(path "/f8ca57fe-b4ec-4658-84e8-4883faa41e21"
 					(reference "M1")
@@
 		)
 		(instances
-			(project "floraflow"
+			(project "bloombot"
 				(path "/f8ca57fe-b4ec-4658-84e8-4883faa41e21"
 					(reference "#PWR015")
@@
 		)
 		(instances
-			(project "floraflow"
+			(project "bloombot"
 				(path "/f8ca57fe-b4ec-4658-84e8-4883faa41e21"
 					(reference "#PWR011")
@@
 		)
 		(instances
-			(project "floraflow"
+			(project "bloombot"
 				(path "/f8ca57fe-b4ec-4658-84e8-4883faa41e21"
 					(reference "U1")
@@
 		)
 		(instances
-			(project "floraflow"
+			(project "bloombot"
 				(path "/f8ca57fe-b4ec-4658-84e8-4883faa41e21"
 					(reference "#PWR010")
